Commit message: 4.6: add regular wheels
- also fixed coordinates for wheel/joint

File: my_robot/urdf/my_robot.xacro (robot description, xacro)
@@ -55,3 +55,66 @@
         </visual>
     </link>
+    <link name="left_wheel">
+        <collision>
+            <origin xyz="0 0 0" rpy=" 0 1.5707 1.5707"/>
+            <geometry>
+                <cylinder radius="0.1" length="0.05"/>
+            </geometry>
+        </collision>
+        <inertial>
+            <mass value="5"/>
+            <origin xyz="0 0 0" rpy=" 0 1.5707 1.5707"/>
+            <inertia
+                ixx="0.1" ixy="0" ixz="0"
+                iyy="0.1" iyz="0"
+                izz="0.1"
+            />
+        </inertial>
+        <visual>
+            <mass value="5"/>
+            <origin xyz="0 0 0" rpy=" 0 1.5707 1.5707"/>
+            <geometry>
+                <cylinder radius="0.1" length="0.05"/>
+            </geometry>
+        </visual>
+    </link>
+     <link name="right_wheel">
+        <collision>
+            <origin xyz="0 0 0" rpy=" 0 1.5707 1.5707"/>
+            <geometry>
+                <cylinder radius="0.1" length="0.05"/>
+            </geometry>
+        </collision>
+        <inertial>
+            <mass value="5"/>
+            <origin xyz="0 0 0" rpy=" 0 1.5707 1.5707"/>
+            <inertia
+                ixx="0.1" ixy="0" ixz="0"
+                iyy="0.1" iyz="0"
+                izz="0.1"
+            />
+        </inertial>
+        <visual>
+            <origin xyz="0 0 0" rpy=" 0 1.5707 1.5707"/>
+            <geometry>
+                <cylinder radius="0.1" length="0.05"/>
+            </geometry>
+        </visual>
+    </link>
+    <joint type="continuous" name="left_wheel_hinge">
+        <origin xyz="0 0.15 0" rpy="0 0 0"/>
+        <child link="left_wheel"/>
+        <parent link="chassis"/>
+        <axis xyz="0 1 0" rpy="0 0 0"/>
+        <limit effort="10000" velocity="1000"/>
+        <dynamics damping="1.0" friction="1.0"/>
+    </joint>
+    <joint type="continuous" name="right_wheel_hinge">
+        <origin xyz="0 -0.15 0" rpy="0 0 0"/>
+        <child link="right_wheel"/>
+        <parent link="chassis"/>
+        <axis xyz="0 1 0" rpy="0 0 0"/>
+        <limit effort="10000" velocity="1000"/>
+        <dynamics damping="1.0" friction="1.0"/>
+    </joint>
 </robot>

Commit message: 4.7 add camera

File: my_robot/urdf/my_robot.xacro (robot description, xacro)
@@ -118,3 +118,33 @@
         <dynamics damping="1.0" friction="1.0"/>
     </joint>
+    <!-- lesson 4.7 add camera -->
+    <link name="camera">
+        <collision>
+            <origin xyz="0 0 0" rpy="0 0 0"/>
+            <geometry>
+                <box size="0.05 0.05 0.05" />
+            </geometry>
+        </collision>
+        <inertial>
+            <origin xyz="0 0 0" rpy="0 0 0"/>
+            <mass   value="0.1"/>
+            <inertia
+                ixx="1e-6" ixy="0" ixz="0"
+                iyy="1e-6" iyz="0"
+                izz="1e-6"
+            />
+        </inertial>
+        <visual>
+            <origin xyz="0 0 0" rpy=" 0 0 0"/>
+            <geometry>
+                <box size="0.05 0.05 0.05" />
+            </geometry>
+        </visual>
+    </link>
+    <joint name="camera_joint" type="fixed">
+        <axis xyz="0 1 0"/>
+        <origin xyz="0.2 0 0" rpy="0 0 0" />
+        <parent link="chassis"/>
+        <child link="camera"/>
+    </joint>
 </robot>

Commit message: 4.7: add lidar
- green color for left wheel as suggested

File: my_robot/urdf/my_robot.xacro (robot description, xacro)
@@ -148,3 +148,37 @@
         <child link="camera"/>
     </joint>
+    <!-- 4.7 add lidar -->
+     <link name="hokuyo">
+        <collision>
+            <origin xyz="0 0 0" rpy="0 0 0"/>
+            <geometry>
+                <box size="0.1 0.1 0.1" />
+            </geometry>
+        </collision>
+        <inertial>
+            <origin xyz="0 0 0" rpy="0 0 0"/>
+            <mass value="1e-5" />
+            <inertia
+                ixx="1e-6" ixy="0" ixz="0"
+                iyy="1e-6" iyz="0"
+                izz="1e-6"
+            />
+        </inertial>
+        <visual>
+            <origin xyz="0 0 0" rpy="0 0 0"/>
+            <geometry>
+                <mesh filename="package://my_robot/meshes/hokuyo.dae" />
+            </geometry>
+        </visual>
+     </link>
+     <joint name="hokuyo_joint" type="fixed">
+        <axis xyz="0 1 0"/>
+        <origin xyz="0.15 0 .1" rpy="0 0 0" />
+        <parent link="chassis"/>
+        <child link="hokuyo"/>
+     </joint>
+     <!-- 4.7 color -->
+     <gazebo reference="left_wheel">
+        <material>Gazebo/Green</material>
+    </gazebo>
 </robot>

Commit message: 4.7 add optional colors?

File: my_robot/urdf/my_robot.xacro (robot description, xacro)
@@ -182,3 +182,12 @@
         <material>Gazebo/Green</material>
     </gazebo>
+    <gazebo reference="right_wheel">
+        <material>Gazebo/Green</material>
+    </gazebo>
+    <gazebo reference="chassis">
+        <material>Gazebo/Blue</material>
+    </gazebo>
+    <gazebo reference="camera">
+        <material>Gazebo/Red</material>
+    </gazebo>
 </robot>

Commit message: 4.17: Update colors per rubric

File: my_robot/urdf/my_robot.xacro (robot description, xacro)
@@ -181,14 +181,17 @@
      <!-- 4.7 color -->
      <gazebo reference="left_wheel">
-        <material>Gazebo/Green</material>
+        <material>Gazebo/SkyBlue</material>
     </gazebo>
     <gazebo reference="right_wheel">
-        <material>Gazebo/Green</material>
+        <material>Gazebo/Orange</material>
     </gazebo>
     <gazebo reference="chassis">
-        <material>Gazebo/Blue</material>
+        <material>Gazebo/Purple</material>
     </gazebo>
     <gazebo reference="camera">
-        <material>Gazebo/Red</material>
+        <material>Gazebo/GreenGlow</material>
+    </gazebo>
+    <gazebo reference="hokuyo">
+        <material>Gzebo/Yellow</material>
     </gazebo>
 </robot>

Commit message: 4.17 update wheel radius and chassis dimensinos per rubric

File: my_robot/urdf/my_robot.xacro (robot description, xacro)
@@ -9,5 +9,5 @@
     </joint>
     <link name='chassis'>
-        <pose>0 0 0.1 0 0 0</pose>
+        <pose>0 0 0.15 0 0 0</pose>
         <inertial>
             <mass value="15.0"/>
@@ -22,5 +22,5 @@
             <origin xyz="0 0 0" rpy=" 0 0 0"/>
             <geometry>
-            <box size=".4 .2 .1"/>
+            <box size=".4 .2 .2"/>
             </geometry>
         </collision>
@@ -28,9 +28,9 @@
             <origin xyz="0 0 0" rpy=" 0 0 0"/>
             <geometry>
-            <box size=".4 .2 .1"/>
+            <box size=".4 .2 .2"/>
             </geometry>
         </visual>
         <collision name='back_caster_collision'>
-            <origin xyz="-0.15 0 -0.05" rpy=" 0 0 0"/>
+            <origin xyz="-0.15 0 -0.10" rpy=" 0 0 0"/>
             <geometry>
             <sphere radius="0.0499"/>
@@ -38,5 +38,5 @@
         </collision>
         <visual name='back_caster_visual'>
-            <origin xyz="-0.15 0 -0.05" rpy=" 0 0 0"/>
+            <origin xyz="-0.15 0 -0.10" rpy=" 0 0 0"/>
             <geometry>
             <sphere radius="0.05"/>
@@ -44,5 +44,5 @@
         </visual>
         <collision name='front_caster_collision'>
-            <origin xyz="0.15 0 -0.05" rpy=" 0 0 0"/>
+            <origin xyz="0.15 0 -0.10" rpy=" 0 0 0"/>
             <geometry>
             <sphere radius="0.0499"/>
@@ -50,5 +50,5 @@
         </collision>
         <visual name='front_caster_visual'>
-            <origin xyz="0.15 0 -0.05" rpy=" 0 0 0"/>
+            <origin xyz="0.15 0 -0.10" rpy=" 0 0 0"/>
             <geometry>
             <sphere radius="0.05"/>
@@ -60,5 +60,5 @@
             <origin xyz="0 0 0" rpy=" 0 1.5707 1.5707"/>
             <geometry>
-                <cylinder radius="0.1" length="0.05"/>
+                <cylinder radius="0.15" length="0.05"/>
             </geometry>
         </collision>
@@ -76,5 +76,5 @@
             <origin xyz="0 0 0" rpy=" 0 1.5707 1.5707"/>
             <geometry>
-                <cylinder radius="0.1" length="0.05"/>
+                <cylinder radius="0.15" length="0.05"/>
             </geometry>
         </visual>
@@ -84,5 +84,5 @@
             <origin xyz="0 0 0" rpy=" 0 1.5707 1.5707"/>
             <geometry>
-                <cylinder radius="0.1" length="0.05"/>
+                <cylinder radius="0.15" length="0.05"/>
             </geometry>
         </collision>
@@ -99,5 +99,5 @@
             <origin xyz="0 0 0" rpy=" 0 1.5707 1.5707"/>
             <geometry>
-                <cylinder radius="0.1" length="0.05"/>
+                <cylinder radius="0.15" length="0.05"/>
             </geometry>
         </visual>
